File: matrix.kicad_sch (KiCad schematic)
At the start: 60 parts, among them SW1 SW_Push, SW10 SW_Push, SW11 SW_Push, SW12 SW_Push, SW13 SW_Push, SW14 SW_Push, SW15 SW_Push, SW16 SW_Push, SW17 SW_Push, SW18 SW_Push, SW19 SW_Push, SW2 SW_Push, SW20 SW_Push, SW21 SW_Push, SW22 SW_Push, SW23 SW_Push, SW24 SW_Push, SW25 SW_Push, SW26 SW_Push, SW27 SW_Push, SW28 SW_Push, SW29 SW_Push, SW3 SW_Push, SW30 SW_Push, SW4 SW_Push, SW5 SW_Push, SW6 SW_Push, SW7 SW_Push, SW8 SW_Push, SW9 SW_Push

Commit message: added routing
Parts:
- D1, D10, D11, D12, D13, D14, D15, D16, D17, D18, D19, D2, D20, D21, D22, D23, D24, D25, D26, D27, D28, D29, D3, D30, D4, D5, D6, D7, D8, D9: footprint Diode_SMD:D_0805_2012Metric -> Diode_SMD:D_SOD-523
Changed lines of the file:
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@@
 			)
 		)
-		(property "Footprint" "Diode_SMD:D_0805_2012Metric"
+		(property "Footprint" "Diode_SMD:D_SOD-523"
 			(at 110.49 106.68 0)
 			(effects
@@
 			)
 		)
-		(property "Datasheet" "~"
+		(property "Datasheet" "BAT54WX-TP"
 			(at 110.49 106.68 0)
 			(effects
@@
 			)
 		)
-		(property "Footprint" "Diode_SMD:D_0805_2012Metric"
+		(property "Footprint" "Diode_SMD:D_SOD-523"
 			(at 95.25 106.68 0)
 			(effects
@@
 			)
 		)
-		(property "Datasheet" "~"
+		(property "Datasheet" "BAT54WX-TP"
 			(at 95.25 106.68 0)
 			(effects
@@
 			)
 		)
-		(property "Footprint" "Diode_SMD:D_0805_2012Metric"
+		(property "Footprint" "Diode_SMD:D_SOD-523"
 			(at 110.49 71.12 0)
 			(effects
@@
 			)
 		)
-		(property "Datasheet" "~"
+		(property "Datasheet" "BAT54WX-TP"
 			(at 110.49 71.12 0)
 			(effects
@@
 			)
 		)
-		(property "Footprint" "Diode_SMD:D_0805_2012Metric"
+		(property "Footprint" "Diode_SMD:D_SOD-523"
 			(at 201.93 88.9 0)
 			(effects
@@
 			)
 		)
-		(property "Datasheet" "~"
+		(property "Datasheet" "BAT54WX-TP"
 			(at 201.93 88.9 0)
 			(effects
@@
 			)
 		)
-		(property "Footprint" "Diode_SMD:D_0805_2012Metric"
+		(property "Footprint" "Diode_SMD:D_SOD-523"
 			(at 171.45 88.9 0)
 			(effects
@@
 			)
 		)
-		(property "Datasheet" "~"
+		(property "Datasheet" "BAT54WX-TP"
 			(at 171.45 88.9 0)
 			(effects
@@
 			)
 		)
-		(property "Footprint" "Diode_SMD:D_0805_2012Metric"
+		(property "Footprint" "Diode_SMD:D_SOD-523"
 			(at 95.25 88.9 0)
 			(effects
@@
 			)
 		)
-		(property "Datasheet" "~"
+		(property "Datasheet" "BAT54WX-TP"
 			(at 95.25 88.9 0)
 			(effects
@@
 			)
 		)
-		(property "Footprint" "Diode_SMD:D_0805_2012Metric"
+		(property "Footprint" "Diode_SMD:D_SOD-523"
 			(at 171.45 106.68 0)
 			(effects
@@
 			)
 		)
-		(property "Datasheet" "~"
+		(property "Datasheet" "BAT54WX-TP"
 			(at 171.45 106.68 0)
 			(effects
@@
 			)
 		)
-		(property "Footprint" "Diode_SMD:D_0805_2012Metric"
+		(property "Footprint" "Diode_SMD:D_SOD-523"
 			(at 140.97 106.68 0)
 			(effects
@@
 			)
 		)
-		(property "Datasheet" "~"
+		(property "Datasheet" "BAT54WX-TP"
 			(at 140.97 106.68 0)
 			(effects
@@
 			)
 		)
-		(property "Footprint" "Diode_SMD:D_0805_2012Metric"
+		(property "Footprint" "Diode_SMD:D_SOD-523"
 			(at 80.01 106.68 0)
 			(effects
@@
 			)
 		)
-		(property "Datasheet" "~"
+		(property "Datasheet" "BAT54WX-TP"
 			(at 80.01 106.68 0)
 			(effects
@@
 			)
 		)
-		(property "Footprint" "Diode_SMD:D_0805_2012Metric"
+		(property "Footprint" "Diode_SMD:D_SOD-523"
 			(at 186.69 106.68 0)
 			(effects
@@
 			)
 		)
-		(property "Datasheet" "~"
+		(property "Datasheet" "BAT54WX-TP"
 			(at 186.69 106.68 0)
 			(effects
@@
 			)
 		)
-		(property "Footprint" "Diode_SMD:D_0805_2012Metric"
+		(property "Footprint" "Diode_SMD:D_SOD-523"
 			(at 156.21 106.68 0)
 			(effects
@@
 			)
 		)
-		(property "Datasheet" "~"
+		(property "Datasheet" "BAT54WX-TP"
 			(at 156.21 106.68 0)
 			(effects
@@
 			)
 		)
-		(property "Footprint" "Diode_SMD:D_0805_2012Metric"
+		(property "Footprint" "Diode_SMD:D_SOD-523"
 			(at 171.45 71.12 0)
 			(effects
@@
 			)
 		)
-		(property "Datasheet" "~"
+		(property "Datasheet" "BAT54WX-TP"
 			(at 171.45 71.12 0)
 			(effects
@@
 			)
 		)
-		(property "Footprint" "Diode_SMD:D_0805_2012Metric"
+		(property "Footprint" "Diode_SMD:D_SOD-523"
 			(at 125.73 71.12 0)
 			(effects
@@
 			)
 		)
-		(property "Datasheet" "~"
+		(property "Datasheet" "BAT54WX-TP"
 			(at 125.73 71.12 0)
 			(effects
@@
 			)
 		)
-		(property "Footprint" "Diode_SMD:D_0805_2012Metric"
+		(property "Footprint" "Diode_SMD:D_SOD-523"
 			(at 140.97 88.9 0)
 			(effects
@@
 			)
 		)
-		(property "Datasheet" "~"
+		(property "Datasheet" "BAT54WX-TP"
 			(at 140.97 88.9 0)
 			(effects
@@
 			)
 		)
-		(property "Footprint" "Diode_SMD:D_0805_2012Metric"
+		(property "Footprint" "Diode_SMD:D_SOD-523"
 			(at 80.01 71.12 0)
 			(effects
@@
 			)
 		)
-		(property "Datasheet" "~"
+		(property "Datasheet" "BAT54WX-TP"
 			(at 80.01 71.12 0)
 			(effects
@@
 			)
 		)
-		(property "Footprint" "Diode_SMD:D_0805_2012Metric"
+		(property "Footprint" "Diode_SMD:D_SOD-523"
 			(at 110.49 88.9 0)
 			(effects
@@
 			)
 		)
-		(property "Datasheet" "~"
+		(property "Datasheet" "BAT54WX-TP"
 			(at 110.49 88.9 0)
 			(effects
@@
 			)
 		)
-		(property "Footprint" "Diode_SMD:D_0805_2012Metric"
+		(property "Footprint" "Diode_SMD:D_SOD-523"
 			(at 201.93 71.12 0)
 			(effects
@@
 			)
 		)
-		(property "Datasheet" "~"
+		(property "Datasheet" "BAT54WX-TP"
 			(at 201.93 71.12 0)
 			(effects
@@
 			)
 		)
-		(property "Footprint" "Diode_SMD:D_0805_2012Metric"
+		(property "Footprint" "Diode_SMD:D_SOD-523"
 			(at 125.73 88.9 0)
 			(effects
@@
 			)
 		)
-		(property "Datasheet" "~"
+		(property "Datasheet" "BAT54WX-TP"
 			(at 125.73 88.9 0)
 			(effects
@@
 			)
 		)
-		(property "Footprint" "Diode_SMD:D_0805_2012Metric"
+		(property "Footprint" "Diode_SMD:D_SOD-523"
 			(at 80.01 88.9 0)
 			(effects
@@
 			)
 		)
-		(property "Datasheet" "~"
+		(property "Datasheet" "BAT54WX-TP"
 			(at 80.01 88.9 0)
 			(effects
@@
 			)
 		)
-		(property "Footprint" "Diode_SMD:D_0805_2012Metric"
+		(property "Footprint" "Diode_SMD:D_SOD-523"
 			(at 95.25 71.12 0)
 			(effects
@@
 			)
 		)
-		(property "Datasheet" "~"
+		(property "Datasheet" "BAT54WX-TP"
 			(at 95.25 71.12 0)
 			(effects
@@
 			)
 		)
-		(property "Footprint" "Diode_SMD:D_0805_2012Metric"
+		(property "Footprint" "Diode_SMD:D_SOD-523"
 			(at 64.77 106.68 0)
 			(effects
@@
 			)
 		)
-		(property "Datasheet" "~"
+		(property "Datasheet" "BAT54WX-TP"
 			(at 64.77 106.68 0)
 			(effects
@@
 			)
 		)
-		(property "Footprint" "Diode_SMD:D_0805_2012Metric"
+		(property "Footprint" "Diode_SMD:D_SOD-523"
 			(at 140.97 71.12 0)
 			(effects
@@
 			)
 		)
-		(property "Datasheet" "~"
+		(property "Datasheet" "BAT54WX-TP"
 			(at 140.97 71.12 0)
 			(effects
@@
 			)
 		)
-		(property "Footprint" "Diode_SMD:D_0805_2012Metric"
+		(property "Footprint" "Diode_SMD:D_SOD-523"
 			(at 156.21 71.12 0)
 			(effects
@@
 			)
 		)
-		(property "Datasheet" "~"
+		(property "Datasheet" "BAT54WX-TP"
 			(at 156.21 71.12 0)
 			(effects
@@
 			)
 		)
-		(property "Footprint" "Diode_SMD:D_0805_2012Metric"
+		(property "Footprint" "Diode_SMD:D_SOD-523"
 			(at 64.77 88.9 0)
 			(effects
@@
 			)
 		)
-		(property "Datasheet" "~"
+		(property "Datasheet" "BAT54WX-TP"
 			(at 64.77 88.9 0)
 			(effects
@@
 			)
 		)
-		(property "Footprint" "Diode_SMD:D_0805_2012Metric"
+		(property "Footprint" "Diode_SMD:D_SOD-523"
 			(at 201.93 106.68 0)
 			(effects
@@
 			)
 		)
-		(property "Datasheet" "~"
+		(property "Datasheet" "BAT54WX-TP"
 			(at 201.93 106.68 0)
 			(effects
@@
 			)
 		)
-		(property "Footprint" "Diode_SMD:D_0805_2012Metric"
+		(property "Footprint" "Diode_SMD:D_SOD-523"
 			(at 186.69 71.12 0)
 			(effects
@@
 			)
 		)
-		(property "Datasheet" "~"
+		(property "Datasheet" "BAT54WX-TP"
 			(at 186.69 71.12 0)
 			(effects
@@
 			)
 		)
-		(property "Footprint" "Diode_SMD:D_0805_2012Metric"
+		(property "Footprint" "Diode_SMD:D_SOD-523"
 			(at 64.77 71.12 0)
 			(effects
@@
 			)
 		)
-		(property "Datasheet" "~"
+		(property "Datasheet" "BAT54WX-TP"
 			(at 64.77 71.12 0)
 			(effects
@@
 			)
 		)
-		(property "Footprint" "Diode_SMD:D_0805_2012Metric"
+		(property "Footprint" "Diode_SMD:D_SOD-523"
 			(at 156.21 88.9 0)
 			(effects
@@
 			)
 		)
-		(property "Datasheet" "~"
+		(property "Datasheet" "BAT54WX-TP"
 			(at 156.21 88.9 0)
 			(effects
@@
 			)
 		)
-		(property "Footprint" "Diode_SMD:D_0805_2012Metric"
+		(property "Footprint" "Diode_SMD:D_SOD-523"
 			(at 125.73 106.68 0)
 			(effects
@@
 			)
 		)
-		(property "Datasheet" "~"
+		(property "Datasheet" "BAT54WX-TP"
 			(at 125.73 106.68 0)
 			(effects
@@
 			)
 		)
-		(property "Footprint" "Diode_SMD:D_0805_2012Metric"
+		(property "Footprint" "Diode_SMD:D_SOD-523"
 			(at 186.69 88.9 0)
 			(effects
@@
 			)
 		)
-		(property "Datasheet" "~"
+		(property "Datasheet" "BAT54WX-TP"
 			(at 186.69 88.9 0)
 			(effects

Commit message: re-done whole pcb
Parts:
- SW1, SW10, SW11, SW12, SW13, SW14, SW15, SW16, SW17, SW18, SW19, SW2, SW20, SW21, SW22, SW23, SW24, SW25, SW26, SW27, SW28, SW29, SW3, SW30, SW4, SW5, SW6, SW7, SW8, SW9: footprint my_switch:SW_Cherry_MX_1.00u_PCB -> my_switch:SW_Cherry_MX_1.00u_PCB_no_support_stems
Changed lines of the file:
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@@
 			)
 		)
-		(property "Footprint" "my_switch:SW_Cherry_MX_1.00u_PCB"
+		(property "Footprint" "my_switch:SW_Cherry_MX_1.00u_PCB_no_support_stems"
 			(at 147.32 78.74 0)
 			(effects
@@
 			)
 		)
-		(property "Footprint" "my_switch:SW_Cherry_MX_1.00u_PCB"
+		(property "Footprint" "my_switch:SW_Cherry_MX_1.00u_PCB_no_support_stems"
 			(at 71.12 78.74 0)
 			(effects
@@
 			)
 		)
-		(property "Footprint" "my_switch:SW_Cherry_MX_1.00u_PCB"
+		(property "Footprint" "my_switch:SW_Cherry_MX_1.00u_PCB_no_support_stems"
 			(at 208.28 96.52 0)
 			(effects
@@
 			)
 		)
-		(property "Footprint" "my_switch:SW_Cherry_MX_1.00u_PCB"
+		(property "Footprint" "my_switch:SW_Cherry_MX_1.00u_PCB_no_support_stems"
 			(at 147.32 60.96 0)
 			(effects
@@
 			)
 		)
-		(property "Footprint" "my_switch:SW_Cherry_MX_1.00u_PCB"
+		(property "Footprint" "my_switch:SW_Cherry_MX_1.00u_PCB_no_support_stems"
 			(at 193.04 60.96 0)
 			(effects
@@
 			)
 		)
-		(property "Footprint" "my_switch:SW_Cherry_MX_1.00u_PCB"
+		(property "Footprint" "my_switch:SW_Cherry_MX_1.00u_PCB_no_support_stems"
 			(at 162.56 78.74 0)
 			(effects
@@
 			)
 		)
-		(property "Footprint" "my_switch:SW_Cherry_MX_1.00u_PCB"
+		(property "Footprint" "my_switch:SW_Cherry_MX_1.00u_PCB_no_support_stems"
 			(at 132.08 96.52 0)
 			(effects
@@
 			)
 		)
-		(property "Footprint" "my_switch:SW_Cherry_MX_1.00u_PCB"
+		(property "Footprint" "my_switch:SW_Cherry_MX_1.00u_PCB_no_support_stems"
 			(at 193.04 78.74 0)
 			(effects
@@
 			)
 		)
-		(property "Footprint" "my_switch:SW_Cherry_MX_1.00u_PCB"
+		(property "Footprint" "my_switch:SW_Cherry_MX_1.00u_PCB_no_support_stems"
 			(at 86.36 96.52 0)
 			(effects
@@
 			)
 		)
-		(property "Footprint" "my_switch:SW_Cherry_MX_1.00u_PCB"
+		(property "Footprint" "my_switch:SW_Cherry_MX_1.00u_PCB_no_support_stems"
 			(at 101.6 96.52 0)
 			(effects
@@
 			)
 		)
-		(property "Footprint" "my_switch:SW_Cherry_MX_1.00u_PCB"
+		(property "Footprint" "my_switch:SW_Cherry_MX_1.00u_PCB_no_support_stems"
 			(at 177.8 96.52 0)
 			(effects
@@
 			)
 		)
-		(property "Footprint" "my_switch:SW_Cherry_MX_1.00u_PCB"
+		(property "Footprint" "my_switch:SW_Cherry_MX_1.00u_PCB_no_support_stems"
 			(at 208.28 78.74 0)
 			(effects
@@
 			)
 		)
-		(property "Footprint" "my_switch:SW_Cherry_MX_1.00u_PCB"
+		(property "Footprint" "my_switch:SW_Cherry_MX_1.00u_PCB_no_support_stems"
 			(at 177.8 78.74 0)
 			(effects
@@
 			)
 		)
-		(property "Footprint" "my_switch:SW_Cherry_MX_1.00u_PCB"
+		(property "Footprint" "my_switch:SW_Cherry_MX_1.00u_PCB_no_support_stems"
 			(at 116.84 60.96 0)
 			(effects
@@
 			)
 		)
-		(property "Footprint" "my_switch:SW_Cherry_MX_1.00u_PCB"
+		(property "Footprint" "my_switch:SW_Cherry_MX_1.00u_PCB_no_support_stems"
 			(at 132.08 60.96 0)
 			(effects
@@
 			)
 		)
-		(property "Footprint" "my_switch:SW_Cherry_MX_1.00u_PCB"
+		(property "Footprint" "my_switch:SW_Cherry_MX_1.00u_PCB_no_support_stems"
 			(at 71.12 60.96 0)
 			(effects
@@
 			)
 		)
-		(property "Footprint" "my_switch:SW_Cherry_MX_1.00u_PCB"
+		(property "Footprint" "my_switch:SW_Cherry_MX_1.00u_PCB_no_support_stems"
 			(at 71.12 96.52 0)
 			(effects
@@
 			)
 		)
-		(property "Footprint" "my_switch:SW_Cherry_MX_1.00u_PCB"
+		(property "Footprint" "my_switch:SW_Cherry_MX_1.00u_PCB_no_support_stems"
 			(at 193.04 96.52 0)
 			(effects
@@
 			)
 		)
-		(property "Footprint" "my_switch:SW_Cherry_MX_1.00u_PCB"
+		(property "Footprint" "my_switch:SW_Cherry_MX_1.00u_PCB_no_support_stems"
 			(at 101.6 78.74 0)
 			(effects
@@
 			)
 		)
-		(property "Footprint" "my_switch:SW_Cherry_MX_1.00u_PCB"
+		(property "Footprint" "my_switch:SW_Cherry_MX_1.00u_PCB_no_support_stems"
 			(at 208.28 60.96 0)
 			(effects
@@
 			)
 		)
-		(property "Footprint" "my_switch:SW_Cherry_MX_1.00u_PCB"
+		(property "Footprint" "my_switch:SW_Cherry_MX_1.00u_PCB_no_support_stems"
 			(at 116.84 96.52 0)
 			(effects
@@
 			)
 		)
-		(property "Footprint" "my_switch:SW_Cherry_MX_1.00u_PCB"
+		(property "Footprint" "my_switch:SW_Cherry_MX_1.00u_PCB_no_support_stems"
 			(at 86.36 78.74 0)
 			(effects
@@
 			)
 		)
-		(property "Footprint" "my_switch:SW_Cherry_MX_1.00u_PCB"
+		(property "Footprint" "my_switch:SW_Cherry_MX_1.00u_PCB_no_support_stems"
 			(at 147.32 96.52 0)
 			(effects
@@
 			)
 		)
-		(property "Footprint" "my_switch:SW_Cherry_MX_1.00u_PCB"
+		(property "Footprint" "my_switch:SW_Cherry_MX_1.00u_PCB_no_support_stems"
 			(at 177.8 60.96 0)
 			(effects
@@
 			)
 		)
-		(property "Footprint" "my_switch:SW_Cherry_MX_1.00u_PCB"
+		(property "Footprint" "my_switch:SW_Cherry_MX_1.00u_PCB_no_support_stems"
 			(at 116.84 78.74 0)
 			(effects
@@
 			)
 		)
-		(property "Footprint" "my_switch:SW_Cherry_MX_1.00u_PCB"
+		(property "Footprint" "my_switch:SW_Cherry_MX_1.00u_PCB_no_support_stems"
 			(at 162.56 96.52 0)
 			(effects
@@
 			)
 		)
-		(property "Footprint" "my_switch:SW_Cherry_MX_1.00u_PCB"
+		(property "Footprint" "my_switch:SW_Cherry_MX_1.00u_PCB_no_support_stems"
 			(at 162.56 60.96 0)
 			(effects
@@
 			)
 		)
-		(property "Footprint" "my_switch:SW_Cherry_MX_1.00u_PCB"
+		(property "Footprint" "my_switch:SW_Cherry_MX_1.00u_PCB_no_support_stems"
 			(at 132.08 78.74 0)
 			(effects
@@
 			)
 		)
-		(property "Footprint" "my_switch:SW_Cherry_MX_1.00u_PCB"
+		(property "Footprint" "my_switch:SW_Cherry_MX_1.00u_PCB_no_support_stems"
 			(at 86.36 60.96 0)
 			(effects
@@
 			)
 		)
-		(property "Footprint" "my_switch:SW_Cherry_MX_1.00u_PCB"
+		(property "Footprint" "my_switch:SW_Cherry_MX_1.00u_PCB_no_support_stems"
 			(at 101.6 60.96 0)
 			(effects

Commit message: added ESD protection, re-wired matrix
Parts:
- D1, D10, D11, D12, D13, D14, D15, D16, D17, D18, D19, D2, D20, D21, D22, D23, D24, D25, D26, D27, D28, D29, D3, D30, D4, D5, D6, D7, D8, D9: footprint Diode_SMD:D_SOD-523 -> Diode_SMD:D_SOD-123
Changed lines of the file:
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@@
 			)
 		)
-		(property "Footprint" "Diode_SMD:D_SOD-523"
+		(property "Footprint" "Diode_SMD:D_SOD-123"
 			(at 110.49 106.68 0)
 			(effects
@@
 			)
 		)
-		(property "Datasheet" "BAT54WX-TP"
+		(property "Datasheet" "621-1N4148W-F"
 			(at 110.49 106.68 0)
 			(effects
@@
 			)
 		)
-		(property "Footprint" "Diode_SMD:D_SOD-523"
+		(property "Footprint" "Diode_SMD:D_SOD-123"
 			(at 95.25 106.68 0)
 			(effects
@@
 			)
 		)
-		(property "Datasheet" "BAT54WX-TP"
+		(property "Datasheet" "621-1N4148W-F"
 			(at 95.25 106.68 0)
 			(effects
@@
 			)
 		)
-		(property "Footprint" "Diode_SMD:D_SOD-523"
+		(property "Footprint" "Diode_SMD:D_SOD-123"
 			(at 110.49 71.12 0)
 			(effects
@@
 			)
 		)
-		(property "Datasheet" "BAT54WX-TP"
+		(property "Datasheet" "621-1N4148W-F"
 			(at 110.49 71.12 0)
 			(effects
@@
 			)
 		)
-		(property "Footprint" "Diode_SMD:D_SOD-523"
+		(property "Footprint" "Diode_SMD:D_SOD-123"
 			(at 201.93 88.9 0)
 			(effects
@@
 			)
 		)
-		(property "Datasheet" "BAT54WX-TP"
+		(property "Datasheet" "621-1N4148W-F"
 			(at 201.93 88.9 0)
 			(effects
@@
 			)
 		)
-		(property "Footprint" "Diode_SMD:D_SOD-523"
+		(property "Footprint" "Diode_SMD:D_SOD-123"
 			(at 171.45 88.9 0)
 			(effects
@@
 			)
 		)
-		(property "Datasheet" "BAT54WX-TP"
+		(property "Datasheet" "621-1N4148W-F"
 			(at 171.45 88.9 0)
 			(effects
@@
 			)
 		)
-		(property "Footprint" "Diode_SMD:D_SOD-523"
+		(property "Footprint" "Diode_SMD:D_SOD-123"
 			(at 95.25 88.9 0)
 			(effects
@@
 			)
 		)
-		(property "Datasheet" "BAT54WX-TP"
+		(property "Datasheet" "621-1N4148W-F"
 			(at 95.25 88.9 0)
 			(effects
@@
 			)
 		)
-		(property "Footprint" "Diode_SMD:D_SOD-523"
+		(property "Footprint" "Diode_SMD:D_SOD-123"
 			(at 171.45 106.68 0)
 			(effects
@@
 			)
 		)
-		(property "Datasheet" "BAT54WX-TP"
+		(property "Datasheet" "621-1N4148W-F"
 			(at 171.45 106.68 0)
 			(effects
@@
 			)
 		)
-		(property "Footprint" "Diode_SMD:D_SOD-523"
+		(property "Footprint" "Diode_SMD:D_SOD-123"
 			(at 140.97 106.68 0)
 			(effects
@@
 			)
 		)
-		(property "Datasheet" "BAT54WX-TP"
+		(property "Datasheet" "621-1N4148W-F"
 			(at 140.97 106.68 0)
 			(effects
@@
 			)
 		)
-		(property "Footprint" "Diode_SMD:D_SOD-523"
+		(property "Footprint" "Diode_SMD:D_SOD-123"
 			(at 80.01 106.68 0)
 			(effects
@@
 			)
 		)
-		(property "Datasheet" "BAT54WX-TP"
+		(property "Datasheet" "621-1N4148W-F"
 			(at 80.01 106.68 0)
 			(effects
@@
 			)
 		)
-		(property "Footprint" "Diode_SMD:D_SOD-523"
+		(property "Footprint" "Diode_SMD:D_SOD-123"
 			(at 186.69 106.68 0)
 			(effects
@@
 			)
 		)
-		(property "Datasheet" "BAT54WX-TP"
+		(property "Datasheet" "621-1N4148W-F"
 			(at 186.69 106.68 0)
 			(effects
@@
 			)
 		)
-		(property "Footprint" "Diode_SMD:D_SOD-523"
+		(property "Footprint" "Diode_SMD:D_SOD-123"
 			(at 156.21 106.68 0)
 			(effects
@@
 			)
 		)
-		(property "Datasheet" "BAT54WX-TP"
+		(property "Datasheet" "621-1N4148W-F"
 			(at 156.21 106.68 0)
 			(effects
@@
 			)
 		)
-		(property "Footprint" "Diode_SMD:D_SOD-523"
+		(property "Footprint" "Diode_SMD:D_SOD-123"
 			(at 171.45 71.12 0)
 			(effects
@@
 			)
 		)
-		(property "Datasheet" "BAT54WX-TP"
+		(property "Datasheet" "621-1N4148W-F"
 			(at 171.45 71.12 0)
 			(effects
@@
 			)
 		)
-		(property "Footprint" "Diode_SMD:D_SOD-523"
+		(property "Footprint" "Diode_SMD:D_SOD-123"
 			(at 125.73 71.12 0)
 			(effects
@@
 			)
 		)
-		(property "Datasheet" "BAT54WX-TP"
+		(property "Datasheet" "621-1N4148W-F"
 			(at 125.73 71.12 0)
 			(effects
@@
 			)
 		)
-		(property "Footprint" "Diode_SMD:D_SOD-523"
+		(property "Footprint" "Diode_SMD:D_SOD-123"
 			(at 140.97 88.9 0)
 			(effects
@@
 			)
 		)
-		(property "Datasheet" "BAT54WX-TP"
+		(property "Datasheet" "621-1N4148W-F"
 			(at 140.97 88.9 0)
 			(effects
@@
 			)
 		)
-		(property "Footprint" "Diode_SMD:D_SOD-523"
+		(property "Footprint" "Diode_SMD:D_SOD-123"
 			(at 80.01 71.12 0)
 			(effects
@@
 			)
 		)
-		(property "Datasheet" "BAT54WX-TP"
+		(property "Datasheet" "621-1N4148W-F"
 			(at 80.01 71.12 0)
 			(effects
@@
 			)
 		)
-		(property "Footprint" "Diode_SMD:D_SOD-523"
+		(property "Footprint" "Diode_SMD:D_SOD-123"
 			(at 110.49 88.9 0)
 			(effects
@@
 			)
 		)
-		(property "Datasheet" "BAT54WX-TP"
+		(property "Datasheet" "621-1N4148W-F"
 			(at 110.49 88.9 0)
 			(effects
@@
 			)
 		)
-		(property "Footprint" "Diode_SMD:D_SOD-523"
+		(property "Footprint" "Diode_SMD:D_SOD-123"
 			(at 201.93 71.12 0)
 			(effects
@@
 			)
 		)
-		(property "Datasheet" "BAT54WX-TP"
+		(property "Datasheet" "621-1N4148W-F"
 			(at 201.93 71.12 0)
 			(effects
@@
 			)
 		)
-		(property "Footprint" "Diode_SMD:D_SOD-523"
+		(property "Footprint" "Diode_SMD:D_SOD-123"
 			(at 125.73 88.9 0)
 			(effects
@@
 			)
 		)
-		(property "Datasheet" "BAT54WX-TP"
+		(property "Datasheet" "621-1N4148W-F"
 			(at 125.73 88.9 0)
 			(effects
@@
 			)
 		)
-		(property "Footprint" "Diode_SMD:D_SOD-523"
+		(property "Footprint" "Diode_SMD:D_SOD-123"
 			(at 80.01 88.9 0)
 			(effects
@@
 			)
 		)
-		(property "Datasheet" "BAT54WX-TP"
+		(property "Datasheet" "621-1N4148W-F"
 			(at 80.01 88.9 0)
 			(effects
@@
 			)
 		)
-		(property "Footprint" "Diode_SMD:D_SOD-523"
+		(property "Footprint" "Diode_SMD:D_SOD-123"
 			(at 95.25 71.12 0)
 			(effects
@@
 			)
 		)
-		(property "Datasheet" "BAT54WX-TP"
+		(property "Datasheet" "621-1N4148W-F"
 			(at 95.25 71.12 0)
 			(effects
@@
 			)
 		)
-		(property "Footprint" "Diode_SMD:D_SOD-523"
+		(property "Footprint" "Diode_SMD:D_SOD-123"
 			(at 64.77 106.68 0)
 			(effects
@@
 			)
 		)
-		(property "Datasheet" "BAT54WX-TP"
+		(property "Datasheet" "621-1N4148W-F"
 			(at 64.77 106.68 0)
 			(effects
@@
 			)
 		)
-		(property "Footprint" "Diode_SMD:D_SOD-523"
+		(property "Footprint" "Diode_SMD:D_SOD-123"
 			(at 140.97 71.12 0)
 			(effects
@@
 			)
 		)
-		(property "Datasheet" "BAT54WX-TP"
+		(property "Datasheet" "621-1N4148W-F"
 			(at 140.97 71.12 0)
 			(effects
@@
 			)
 		)
-		(property "Footprint" "Diode_SMD:D_SOD-523"
+		(property "Footprint" "Diode_SMD:D_SOD-123"
 			(at 156.21 71.12 0)
 			(effects
@@
 			)
 		)
-		(property "Datasheet" "BAT54WX-TP"
+		(property "Datasheet" "621-1N4148W-F"
 			(at 156.21 71.12 0)
 			(effects
@@
 			)
 		)
-		(property "Footprint" "Diode_SMD:D_SOD-523"
+		(property "Footprint" "Diode_SMD:D_SOD-123"
 			(at 64.77 88.9 0)
 			(effects
@@
 			)
 		)
-		(property "Datasheet" "BAT54WX-TP"
+		(property "Datasheet" "621-1N4148W-F"
 			(at 64.77 88.9 0)
 			(effects
@@
 			)
 		)
-		(property "Footprint" "Diode_SMD:D_SOD-523"
+		(property "Footprint" "Diode_SMD:D_SOD-123"
 			(at 201.93 106.68 0)
 			(effects
@@
 			)
 		)
-		(property "Datasheet" "BAT54WX-TP"
+		(property "Datasheet" "621-1N4148W-F"
 			(at 201.93 106.68 0)
 			(effects
@@
 			)
 		)
-		(property "Footprint" "Diode_SMD:D_SOD-523"
+		(property "Footprint" "Diode_SMD:D_SOD-123"
 			(at 186.69 71.12 0)
 			(effects
@@
 			)
 		)
-		(property "Datasheet" "BAT54WX-TP"
+		(property "Datasheet" "621-1N4148W-F"
 			(at 186.69 71.12 0)
 			(effects
@@
 			)
 		)
-		(property "Footprint" "Diode_SMD:D_SOD-523"
+		(property "Footprint" "Diode_SMD:D_SOD-123"
 			(at 64.77 71.12 0)
 			(effects
@@
 			)
 		)
-		(property "Datasheet" "BAT54WX-TP"
+		(property "Datasheet" "621-1N4148W-F"
 			(at 64.77 71.12 0)
 			(effects
@@
 			)
 		)
-		(property "Footprint" "Diode_SMD:D_SOD-523"
+		(property "Footprint" "Diode_SMD:D_SOD-123"
 			(at 156.21 88.9 0)
 			(effects
@@
 			)
 		)
-		(property "Datasheet" "BAT54WX-TP"
+		(property "Datasheet" "621-1N4148W-F"
 			(at 156.21 88.9 0)
 			(effects
@@
 			)
 		)
-		(property "Footprint" "Diode_SMD:D_SOD-523"
+		(property "Footprint" "Diode_SMD:D_SOD-123"
 			(at 125.73 106.68 0)
 			(effects
@@
 			)
 		)
-		(property "Datasheet" "BAT54WX-TP"
+		(property "Datasheet" "621-1N4148W-F"
 			(at 125.73 106.68 0)
 			(effects
@@
 			)
 		)
-		(property "Footprint" "Diode_SMD:D_SOD-523"
+		(property "Footprint" "Diode_SMD:D_SOD-123"
 			(at 186.69 88.9 0)
 			(effects
@@
 			)
 		)
-		(property "Datasheet" "BAT54WX-TP"
+		(property "Datasheet" "621-1N4148W-F"
 			(at 186.69 88.9 0)
 			(effects
